File: sii151.kicad_pcb (KiCad board)
At the start: 4 copper layers, 28.2 x 57.8 mm, 37 parts, among them J101 HDMI_A, J102 Conn_01x40, U101 Sii151, U102 24LC02

Commit message: wip
Routing:
- net +3V3: track 51.1 -> 57.0 mm

Commit message: Rev.A ordered
Parts:
- removed 100n104: C_Small, Capacitor_SMD:C_0402_1005Metric
- removed 1u102: C_Small, Capacitor_SMD:C_0603_1608Metric
- removed the R103 at (141.3, 21.6)
- removed the U102 at (142.2, 26.7)
- added C103: 1u, Capacitor_SMD:C_0603_1608Metric, F.Cu at (122.0, 47.6)
- added C104: 100n, Capacitor_SMD:C_0402_1005Metric, F.Cu at (120.5, 38.7)
- added J103: Conn_01x04, Connector_PinHeader_2.00mm:PinHeader_1x04_P2.00mm_Vertical, F.Cu at (143.8, 21.3)
- added J104: Conn_01x02, Connector_PinHeader_2.54mm:PinHeader_1x02_P2.54mm_Vertical, F.Cu at (119.0, 55.0)
- added JP105: SolderJumper_2_Bridged, Jumper:SolderJumper-2_P1.3mm_Bridged_RoundedPad1.0x1.5mm, B.Cu at (128.6, 44.2)
- added R101: 47k, Resistor_SMD:R_0402_1005Metric, F.Cu at (144.0, 24.6)
- added REF**: OSHW-Symbol_6.7x6mm_SilkScreen, Symbol:OSHW-Symbol_6.7x6mm_SilkScreen, F.Cu at (120.7, 17.9)
- added U101: 24LC02, Package_SO:SO-8_3.9x4.9mm_P1.27mm, F.Cu at (142.0, 30.1)
- C101: renamed from 100n101; value C_Small -> 100n
- C102: renamed from 100n102; value C_Small -> 100n
- C105: renamed from 100n105; value C_Small -> 100n
- C106: renamed from 100n106; value C_Small -> 100n
- C107: renamed from 1u101; value C_Small -> 1u
- C108: renamed from 100n109; value C_Small -> 100n
- C109: renamed from 100n110; value C_Small -> 100n
- C110: renamed from 100n107; value C_Small -> 100n
- C111: renamed from 100n108; value C_Small -> 100n
- C112: renamed from 100n103; value C_Small -> 100n
- C113: renamed from 1u103; value C_Small -> 1u
- moved J101 4.95 mm to (132.4, 21.5)
- moved R102 3.52 mm to (141.6, 24.6), turned to 180 degrees
- renumbered JP102 to JP101, JP103 to JP102, JP104 to JP103, JP101 to JP104, L103 to L101, L101 to L102, L102 to L103, R106 to R103, R101 to R104, R104 to R105, R105 to R106, RN102 to RN101, RN103 to RN102, RN104 to RN103, RN105 to RN104, RN101 to RN105, U101 to U102
Connections:
- R102 pad 1: Net-(J101-Pad16) -> Net-(J101-Pad15)
- U102 pad 8: Net-(U101-Pad8) -> Net-(JP105-Pad2)
- U102 pad 9: Net-(U101-Pad8) -> Net-(JP105-Pad1)
Routing:
- net Net-(J101-Pad15): track 7.80 -> 25.7 mm, vias 0 -> 1
- net Net-(J101-Pad16): track 8.50 -> 23.4 mm, vias 0 -> 1
- net Net-(JP105-Pad1): track 0.00 -> 6.44 mm, vias 0 -> 1
- net /RX1+: track 58.2 -> 52.9 mm
- net /RX1-: track 58.2 -> 53.3 mm
- net /RX2+: track 58.2 -> 53.5 mm
- net /RX2-: track 58.2 -> 53.6 mm
- net /RX0+: track 58.2 -> 54.1 mm
- net /RX0-: track 58.2 -> 54.1 mm
- net /RXC-: track 58.2 -> 54.1 mm
- net /RXC+: track 58.3 -> 54.2 mm
- net Net-(JP105-Pad2): track 0.00 -> 3.91 mm, vias 0 -> 1
- net Net-(J101-Pad18): track 18.4 -> 21.5 mm, vias 3 -> 0
- net Net-(JP102-Pad2): track 11.5 -> 13.6 mm
- net Net-(JP101-Pad2): track 13.7 -> 12.9 mm
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Other:
- board size 28.2 x 57.8 mm -> 28.2 x 55 mm
- net class HDMI: trace_width 0.2 -> 0.127
- rule trace_min: 0.2 -> 0.127
- board text added: "(c) Georg Ottinger 2020"
- board text added: "+3V3"
- board text added: "CC BY-SA 3.0"
- board text added: "DFO"
- board text added: "DPS"
- board text added: "GND"
- board text added: "OCK_INV"
- board text added: "PDO_SCDT"
- board text added: "SCL"
- board text added: "SDA"
- board text added: "SII151 HDMI->TFT Adapter Rev.A"
- board text added: "ST"
- board text added: "V+"

Commit message: Rev.A
Parts:
- removed RN104: 47, Resistor_SMD:R_Array_Convex_4x0402
- added R109: 47, Resistor_SMD:R_0402_1005Metric, F.Cu at (139.1, 50.3)
- added R110: 47, Resistor_SMD:R_0402_1005Metric, F.Cu at (140.2, 50.3)
- added R111: 47, Resistor_SMD:R_0402_1005Metric, F.Cu at (125.5, 50.8)
- added R112: 47, Resistor_SMD:R_0402_1005Metric, F.Cu at (126.5, 50.8)
- J102: footprint Connector_FFC-FPC:TE_4-1734839-0_1x40-1MP_P0.5mm_Horizontal -> lib:TE_4-1734839-0_1x40-1MP_P0.5mm_Horizontal
- moved RN101 14.3 mm to (137.4, 50.3)
- moved RN102 6.42 mm to (123.7, 50.8)
- moved R107 4.75 mm to (134.1, 53.6)
- moved R108 4.73 mm to (135.1, 53.6)
- moved RN103 3.95 mm to (129.9, 52.8)
- moved C111 0.64 mm to (128.0, 50.4)
- moved REF** 0.40 mm to (120.8, 18.3)
Connections:
- J101 pad 11: Net-(J101-Pad11) -> GND
- J101 pad 2: Net-(J101-Pad2) -> GND
- J101 pad 5: Net-(J101-Pad5) -> GND
- J101 pad 8: Net-(J101-Pad8) -> GND
- R107 pad 1: Net-(J102-Pad34) -> Net-(J102-Pad24)
- R108 pad 1: Net-(J102-Pad35) -> Net-(J102-Pad25)
- RN102 pad 5: Net-(J102-Pad14) -> Net-(J102-Pad29)
- RN102 pad 6: Net-(J102-Pad15) -> Net-(J102-Pad30)
- RN102 pad 7: Net-(J102-Pad19) -> Net-(J102-Pad31)
- RN102 pad 8: Net-(J102-Pad20) -> Net-(J102-Pad33)
- RN103 pad 5: Net-(J102-Pad21) -> Net-(J102-Pad19)
- RN103 pad 6: Net-(J102-Pad23) -> Net-(J102-Pad20)
- RN103 pad 7: Net-(J102-Pad24) -> Net-(J102-Pad21)
- RN103 pad 8: Net-(J102-Pad25) -> Net-(J102-Pad23)
- U102 pad 12: Net-(RN101-Pad4) -> Net-(RN102-Pad4)
- U102 pad 13: Net-(RN101-Pad3) -> Net-(RN102-Pad3)
- U102 pad 14: Net-(RN101-Pad2) -> Net-(RN102-Pad2)
- U102 pad 15: Net-(RN101-Pad1) -> Net-(RN102-Pad1)
- U102 pad 16: Net-(RN102-Pad4) -> Net-(R111-Pad2)
- U102 pad 17: Net-(RN102-Pad3) -> Net-(R112-Pad2)
- U102 pad 22: Net-(RN102-Pad2) -> Net-(RN103-Pad4)
- U102 pad 23: Net-(RN102-Pad1) -> Net-(RN103-Pad3)
- U102 pad 24: Net-(RN103-Pad4) -> Net-(RN103-Pad2)
- U102 pad 25: Net-(RN103-Pad3) -> Net-(RN103-Pad1)
- U102 pad 26: Net-(RN103-Pad2) -> Net-(R107-Pad2)
- U102 pad 27: Net-(RN103-Pad1) -> Net-(R108-Pad2)
- U102 pad 32: Net-(RN104-Pad4) -> Net-(RN101-Pad4)
- U102 pad 33: Net-(RN104-Pad3) -> Net-(RN101-Pad3)
- U102 pad 34: Net-(RN104-Pad2) -> Net-(RN101-Pad2)
- U102 pad 35: Net-(RN104-Pad1) -> Net-(RN101-Pad1)
- U102 pad 36: Net-(R107-Pad2) -> Net-(R109-Pad2)
- U102 pad 37: Net-(R108-Pad2) -> Net-(R110-Pad2)
Routing:
- net Net-(J102-Pad15): track 3.60 -> 23.5 mm, vias 0 -> 2
- net Net-(J102-Pad9): track 4.30 -> 23.3 mm, vias 0 -> 2
- net Net-(J102-Pad11): track 4.31 -> 23.1 mm, vias 0 -> 2
- net Net-(J102-Pad10): track 4.30 -> 22.8 mm, vias 0 -> 2
- net Net-(J102-Pad13): track 4.32 -> 22.6 mm, vias 0 -> 2
- net Net-(J102-Pad14): track 3.60 -> 21.0 mm, vias 0 -> 2
- net Net-(J102-Pad33): track 3.22 -> 19.3 mm
- net Net-(J102-Pad34): track 3.09 -> 19.2 mm
- net Net-(J102-Pad35): track 3.30 -> 19.0 mm
- net Net-(J102-Pad31): track 3.08 -> 18.7 mm
- net Net-(J102-Pad30): track 3.27 -> 18.3 mm
- net Net-(J102-Pad29): track 3.31 -> 18.0 mm
- net GND: track 97.0 -> 107.4 mm, vias 36 -> 39
- net Net-(RN101-Pad4): track 10.8 -> 1.88 mm
- net Net-(J102-Pad23): track 3.26 -> 11.9 mm, vias 0 -> 2
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
Commit message: Rev.B
Parts:
- removed REF**: OSHW-Symbol_6.7x6mm_SilkScreen, Symbol:OSHW-Symbol_6.7x6mm_SilkScreen
- added C114: 100n, Capacitor_SMD:C_0402_1005Metric, F.Cu at (138.0, 30.1)
- added C115: 1u, Capacitor_SMD:C_0603_1608Metric, B.Cu at (122.4, 51.4)
- added R113: 1k, Resistor_SMD:R_0402_1005Metric, F.Cu at (139.5, 24.6)
- added U103: LD1117S33TR_SOT223, Package_TO_SOT_SMD:SOT-223-3_TabPin2, B.Cu at (121.0, 46.3)
- J104: value Conn_01x02 -> Conn_01x03; footprint Connector_PinHeader_2.54mm:PinHeader_1x02_P2.54mm_Vertical -> Connector_PinHeader_2.54mm:PinHeader_1x03_P2.54mm_Vertical
- moved J104 2.54 mm to (118.9, 57.5), turned to 180 degrees
- moved R103 0.29 mm to (121.8, 52.5)
Connections:
- net Net-(J101-Pad18) renamed VBUS
- C113 pad 1: +3V3 -> +5V
- J102 pad 39: +3V3 -> +5V
- J102 pad 40: +3V3 -> +5V
- J104 pad 1: +3V3 -> +5V
- J104 pad 2: GND -> SYNC_DET
- JP104 pad 3: +3V3 -> +5V
- JP105 pad 2: Net-(JP105-Pad2) -> SYNC_DET
- RN105 pad 7: Net-(J102-Pad4) -> Net-(J102-Pad5)
- RN105 pad 8: Net-(J102-Pad5) -> Net-(J102-Pad4)
- U102 pad 8: Net-(JP105-Pad2) -> SYNC_DET
Routing:
- net +5V: track 0.00 -> 61.7 mm, vias 0 -> 4
- net SYNC_DET: track 0.00 -> 20.0 mm, vias 0 -> 1
- net GND: track 107.4 -> 116.3 mm, vias 39 -> 38
- net Net-(J101-Pad19): track 0.00 -> 4.70 mm
- net VBUS: track 21.5 -> 26.1 mm
- net Net-(JP105-Pad2): track 3.91 -> 0.00 mm, vias 1 -> 0
- net +3V3: track 58.6 -> 55.7 mm, vias 15 -> 12
- net Net-(J102-Pad4): track 25.8 -> 28.5 mm
- net Net-(J102-Pad5): track 26.2 -> 24.8 mm
- net Net-(J102-Pad2): track 24.0 -> 23.2 mm
- net Net-(J102-Pad9): track 23.3 -> 22.5 mm
- net Net-(J102-Pad10): track 22.8 -> 22.1 mm
- net Net-(J102-Pad11): track 23.1 -> 22.4 mm
Other:
- net class Power added: clearance 0.2, trace_width 0.5, via_dia 0.8, via_drill 0.4
- board text added: "+5V"
- board text added: "SII151 HDMI->TFT Adapter Rev.B"
- board text added: "SYNCED"
- board text removed: "+3V3"
- board text removed: "SII151 HDMI->TFT Adapter Rev.A"
