File: sii151.sch (KiCad schematic (older format))
At the start: 37 parts, among them J101 HDMI_A, J102 Conn_01x40, U101 Sii151, U102 24LC02

Commit message: Rev.A ordered
Parts:
- added J103: Conn_01x04, Connector_PinHeader_2.00mm:PinHeader_1x04_P2.00mm_Vertical, symbol Connector_Generic:Conn_01x04
- added J104: Conn_01x02, Connector_PinHeader_2.54mm:PinHeader_1x02_P2.54mm_Vertical, symbol Connector_Generic:Conn_01x02
- added JP105: SolderJumper_2_Bridged, Jumper:SolderJumper-2_P1.3mm_Bridged_RoundedPad1.0x1.5mm, symbol Jumper:SolderJumper_2_Bridged
- C101: renamed from 100n101; value C_Small -> 100n
- C102: renamed from 100n102; value C_Small -> 100n
- C103: renamed from 1u102; value C_Small -> 1u
- C104: renamed from 100n104; value C_Small -> 100n
- C105: renamed from 100n105; value C_Small -> 100n
- C106: renamed from 100n106; value C_Small -> 100n
- C107: renamed from 1u101; value C_Small -> 1u
- C108: renamed from 100n109; value C_Small -> 100n
- C109: renamed from 100n110; value C_Small -> 100n
- C110: renamed from 100n107; value C_Small -> 100n
- C111: renamed from 100n108; value C_Small -> 100n
- C112: renamed from 100n103; value C_Small -> 100n
- C113: renamed from 1u103; value C_Small -> 1u
- renumbered JP102 to JP101, JP103 to JP102, JP104 to JP103, JP101 to JP104, L103 to L101, L101 to L102, L102 to L103, R102 to R101, R103 to R102, R106 to R103, R101 to R104, R104 to R105, R105 to R106, RN102 to RN101, RN103 to RN102, RN104 to RN103, RN105 to RN104, RN101 to RN105, U102 to U101, U101 to U102
Connections:
- net +3V3: now also J104.1 (Pin_1)
- net GND: now also J103.4 (Pin_4), J104.2 (Pin_2)
- net at U102.8 (SCDT): now also JP105.2 (B); no longer U102.9 (PDO)
- net at J101.15 (SCL), R102.1, U101.6 (SCL): now also J103.3 (Pin_3)
- net at J101.16 (SDA), R101.1, U101.5 (SDA): now also J103.2 (Pin_2)
- net at J101.18 (+5V), R101.2, R102.2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: now also J103.1 (Pin_1)
- new net: JP105.1 (A), U102.9 (PDO)

Commit message: Rev.A
Parts:
- removed RN104: 47, Resistor_SMD:R_Array_Convex_4x0402, symbol Device:R_Pack04
- added R109, R110, R111, R112: 47, Resistor_SMD:R_0402_1005Metric, symbol Device:R
- J102: footprint Connector_FFC-FPC:TE_4-1734839-0_1x40-1MP_P0.5mm_Horizontal -> lib:TE_4-1734839-0_1x40-1MP_P0.5mm_Horizontal
Connections:
- net GND: now also J101.11 (CKS), J101.2 (D2S), J101.5 (D1S), J101.8 (D0S)
- net at J102.14 (Pin_14): now also R109.1; no longer RN102.5 (R4.2)
- net at J102.15 (Pin_15): now also R110.1; no longer RN102.6 (R3.2)
- net at J102.19 (Pin_19): now also RN103.5 (R4.2); no longer RN102.7 (R2.2)
- net at J102.20 (Pin_20): now also RN103.6 (R3.2); no longer RN102.8 (R1.2)
- net at J102.21 (Pin_21): now also RN103.7 (R2.2); no longer RN103.5 (R4.2)
- net at J102.23 (Pin_23): now also RN103.8 (R1.2); no longer RN103.6 (R3.2)
- net at J102.24 (Pin_24): now also R107.1; no longer RN103.7 (R2.2)
- net at J102.25 (Pin_25): now also R108.1; no longer RN103.8 (R1.2)
- net at J102.29 (Pin_29): now also RN102.5 (R4.2)
- net at J102.30 (Pin_30): now also RN102.6 (R3.2)
- net at J102.31 (Pin_31): now also RN102.7 (R2.2)
- net at J102.33 (Pin_33): now also RN102.8 (R1.2)
- net at J102.34 (Pin_34): now also R111.1; no longer R107.1
- net at J102.35 (Pin_35): now also R112.1; no longer R108.1
- net at U102.12 (QE2): now also RN102.4 (R4.1)
- net at U102.13 (QE3): now also RN102.3 (R3.1)
- net at U102.14 (QE4): now also RN102.2 (R2.1)
- net at U102.15 (QE5): now also RN102.1 (R1.1)
- net at U102.16 (QE6): now also R111.2; no longer R107.2
- net at U102.17 (QE7): now also R112.2; no longer R108.2
- net at U102.22 (QE10): now also RN103.4 (R4.1); no longer RN102.2 (R2.1)
- net at U102.23 (QE11): now also RN103.3 (R3.1); no longer RN102.1 (R1.1)
- net at U102.24 (QE12): now also RN103.2 (R2.1); no longer RN103.4 (R4.1)
- net at U102.25 (QE13): now also RN103.1 (R1.1); no longer RN103.3 (R3.1)
- net at U102.26 (QE14): now also R107.2; no longer RN103.2 (R2.1)
- net at U102.27 (QE15): now also R108.2; no longer RN103.1 (R1.1)
- net at U102.36 (QE22): now also R109.2; no longer RN102.4 (R4.1)
- net at U102.37 (QE23): now also R110.2; no longer RN102.3 (R3.1)
Other:
- moved on the sheet: R107, R108, RN103

Commit message: Rev.B
Parts:
- added C114: 100n, Capacitor_SMD:C_0402_1005Metric, symbol Device:C_Small
- added C115: 1u, Capacitor_SMD:C_0603_1608Metric, symbol Device:C_Small
- added R113: 1k, Resistor_SMD:R_0402_1005Metric, symbol Device:R
- added U103: LD1117S33TR_SOT223, Package_TO_SOT_SMD:SOT-223-3_TabPin2, symbol Regulator_Linear:LD1117S33TR_SOT223
- J104: value Conn_01x02 -> Conn_01x03; footprint Connector_PinHeader_2.54mm:PinHeader_1x02_P2.54mm_Vertical -> Connector_PinHeader_2.54mm:PinHeader_1x03_P2.54mm_Vertical; symbol Connector_Generic:Conn_01x02 -> Connector_Generic:Conn_01x03
Connections:
- net +3V3: now also U103.2 (VO); no longer C113.1, J102.39 (Pin_39), J102.40 (Pin_40), J104.1 (Pin_1), JP104.3 (B)
- net GND: now also J104.3 (Pin_3), C114.2, C115.2, U103.1 (GND); no longer J104.2 (Pin_2)
- net at J102.4 (Pin_4): now also RN105.8 (R1.2); no longer RN105.7 (R2.2)
- net at J102.5 (Pin_5): now also RN105.7 (R2.2); no longer RN105.8 (R1.2)
- net SYNC_DET: now reaches JP105.2 (B), U102.8 (SCDT)
- net SYNC_DET: now also J104.2 (Pin_2)
- net VBUS: now reaches J101.18 (+5V), J103.1 (Pin_1), R101.2, R102.2, U101.8 (VCC)
- net VBUS: now also C114.1, R113.2
- net at J101.19 (HPD): now also R113.1
- new net +5V: C113.1, C115.1, J102.39 (Pin_39), J102.40 (Pin_40), J104.1 (Pin_1), JP104.3 (B), U103.3 (VI)
Other:
- moved on the sheet: J103, JP105, R101, R102, U101
